File: CircuitDiagrams/IlMattoCamera/cameras.brd (EAGLE design)
At the start: 100 x 80 mm, 19 parts, among them Q1 12MHz, U1 ATMEGA644-20PU, X1 SDBMF

Commit message: Finished Circuit Diagram of Il Matto Camera Platform
Parts:
- added C3, C4: 22pF, resistor:C025-040X050
- added CAM0, CAM1: OV7670, seblov:OV7670
- added D1, D2, D3, D4, D5, D6, D7, D8, D9: U57X32, led:U57X32
- added Q2: 12MHz, crystal:HC49/S
- added R11, R12, R13, R14, R15: 10k, resistor:0204/7
- added R16: 330, resistor:0204/7
- added R17, R18, R19, R20: 68, resistor:0204/7
- added R21, R22: 1k5, resistor:0204/7
- added S2, S3, S4, S5, S6: (no value), SparkFun:TACTILE-PTH
- added U3: PCA9542A, seblov:TSSOP14
- R1: value (none) -> 10k
- U$1, U$2: value OV7670 -> ISP; device seblov:OV7670 -> seblov:DUALHEAD_TH_6
- U$3: value PCA9542A -> MEGA168; device seblov:TSSOP14 -> seblov:MEGA168
- moved U$1 239.3 mm to (-168.9, -182.9)
- moved U$2 238.7 mm to (-176.5, -182.9)
- moved U$3 199.5 mm to (-186.7, -158.8)
Connections:
- net N$10 renamed XTAL2
- net PB2 renamed 644_PB2
- net PB3 renamed 644_PB3
- net PD0 renamed 644_PD0
- net PD1 renamed 644_PD1
- removed net N$2: R1.1, S1.3, S1.4, U1.9
- removed net N$3: R6.2, U$3.9
- removed net N$4: R7.2, U$3.10
- removed net N$6: R9.2, U$3.5
- removed net N$7: R10.2, U$3.6
- removed net N$9: C1.2, C2.2
- removed net PB0: U1.1, X1.SW2
- removed net PB1: U1.2, X1.SW1
- removed net PB4: U1.5, X1.1
- removed net PB5: U1.6, X1.2
- removed net PB6: U1.7, X1.7
- removed net PB7: U1.8, X1.5
- removed net PC2: U$2.RCLK, U1.24
- removed net PC3: U$2.RRST, U1.25
- removed net PC4: U$2.WEN, U1.26
- removed net PC5: U$2.WRST, U1.27
- removed net PC6: U$1.NOE, U1.28
- removed net PC7: U$2.NOE, U1.29
- removed net PD2: U$1.VSYNC, U1.16
- removed net PD3: U$2.VSYNC, U1.17
- removed net PD4: U$1.RCLK, U1.18
- removed net PD5: U$1.RRST, U1.19
- removed net PD6: U$1.WEN, U1.20
- removed net PD7: U$1.WRST, U1.21
- new net 168RESET: R11.1, S2.3, S2.4, U$2.5, U$3.PC6(NRESET)
- new net 168_PB3: U$2.4, U$3.PB3(MOSI/OC2A)
- new net 168_PB4: U$2.1, U$3.PB4(MISO)
- new net 168_PB5: U$2.3, U$3.PB5(SCK)
- new net 168_PB6: C4.1, Q2.1, U$3.PB6(OSC1)
- new net 168_PB7: C3.1, Q2.2, U$3.PB7(OSC2)
- new net 168_PC0: R12.1, S3.3, S3.4, U$3.PC0(ADC0)
- new net 168_PC1: R13.1, S4.3, S4.4, U$3.PC1(ADC1)
- new net 168_PC2: R14.1, S5.3, S5.4, U$3.PC2(ADC2)
- new net 168_PC3: R15.1, S6.3, S6.4, U$3.PC3(ADC3)
- new net 168_PD0: D1.A, U$3.PD0(RXD)
- new net 168_PD1: D2.A, U$3.PD1(TXD)
- new net 168_PD2: D3.A, U$3.PD2(INT0)
- new net 168_PD3: D4.A, U$3.PD3(INT1)
- new net 168_PD4: D5.A, U$3.PD4
- new net 168_PD5: D6.A, U$3.PD5(OC0B)
- new net 168_PD6: D7.A, U$3.PD6(OC0A)
- new net 168_PD7: D8.A, U$3.PD7
- new net 644RESET: R1.1, S1.3, S1.4, U$1.5, U1.9
- new net 644_MISO: R20.1, U$1.1, U1.7
- new net 644_MOSI: R18.1, U$1.4, U1.6
- new net 644_NSS: R17.1, U1.5
- new net 644_SCLK: R19.1, U$1.3, U1.8
- new net N$13: R17.2, X1.1
- new net N$27: R18.2, X1.2
- new net N$28: D9.A, R16.1
- new net N$29: R19.2, X1.5
- new net N$30: R20.2, X1.7
- new net N$31: R21.2, X1.SW1
- new net N$32: R22.2, X1.SW2
- new net NOE0: CAM0.NOE, U1.28
- new net NOE1: CAM1.NOE, U1.29
- new net RCL1: CAM1.RCLK, U1.24
- new net RCLK0: CAM0.RCLK, U1.18
- new net RRST0: CAM0.RRST, U1.19
- new net RRST1: CAM1.RRST, U1.25
- new net SCL0: CAM0.SCL, R10.2, U3.6
- new net SCL1: CAM1.SCL, R7.2, U3.10
- new net SDA0: CAM0.SDA, R9.2, U3.5
- new net SDA1: CAM1.SDA, R6.2, U3.9
- new net SDCD: R21.1, U1.2
- new net SDWP: R22.1, U1.1
- new net VSYNC1: CAM1.VSYNC, U1.17
- new net VYNC0: CAM0.VSYNC, U1.16
- new net WEN0: CAM0.WEN, U1.20
- new net WEN1: CAM1.WEN, U1.26
- new net WRST0: CAM0.WRST, U1.21
- new net WRST1: CAM1.WRST, U1.27
- net +3V3: now also CAM0.3V3, CAM1.3V3, R11.2, R12.2, R13.2, R14.2, R15.2, R16.2, U$1.2, U$2.2, U$3.AREF, U$3.AVCC, U$3.VCC, U3.1, U3.14; no longer U$1.3V3, U$2.3V3, U$3.1, U$3.14
- net GND: now also C1.2, C2.2, C3.2, C4.2, CAM0.GND, CAM0.GND2, CAM1.GND, CAM1.GND2, D1.K, D2.K, D3.K, D4.K, D5.K, D6.K, D7.K, D8.K, D9.K, S2.1, S2.2, S3.1, S3.2, S4.1, S4.2, S5.1, S5.2, S6.1, S6.2, U$1.6, U$2.6, U$3.AGND, U$3.GND, U3.2, U3.3, U3.7, X1.SW3; no longer U$1.GND, U$1.GND2, U$2.GND, U$2.GND2, U$3.2, U$3.3, U$3.7
- net N$1: now also U3.8; no longer U$3.8
- net N$5: now also U3.4; no longer U$3.4
- net N$8: now also U3.11; no longer U$3.11
- net OVDATA0: now also CAM0.D0, CAM1.D0; no longer U$1.D0, U$2.D0
- net OVDATA1: now also CAM0.D1, CAM1.D1; no longer U$1.D1, U$2.D1
- net OVDATA2: now also CAM0.D2, CAM1.D2; no longer U$1.D2, U$2.D2
- net OVDATA3: now also CAM0.D3, CAM1.D3; no longer U$1.D3, U$2.D3
- net OVDATA4: now also CAM0.D4, CAM1.D4; no longer U$1.D4, U$2.D4
- net OVDATA5: now also CAM0.D5, CAM1.D5; no longer U$1.D5, U$2.D5
- net OVDATA6: now also CAM0.D6, CAM1.D6; no longer U$1.D6, U$2.D6
- net OVDATA7: now also CAM0.D7, CAM1.D7; no longer U$1.D7, U$2.D7
- net SCL: now also U$3.PC5(ADC5), U3.12; no longer U$1.SCL, U$2.SCL, U$3.12
- net SDA: now also U$3.PC4(ADC4), U3.13; no longer U$1.SDA, U$2.SDA, U$3.13
Other:
- board size 100 x 80 mm -> 93.7 x 80 mm
