File: CircuitDiagrams/Project/project.sch (EAGLE design)
At the start: 124 parts, among them IC1 UC3C, IC2 PCA9542A, IC3 MT48LC4M16A2TSOP54, IC4 TB6593FNGSSOP20, IC5 TB6593FNGSSOP20, J1 JTAG2.54MM2X5TH, J2 1BY2THROUGHHOLE, J3 1BY2THROUGHHOLE, J4 1BY2THROUGHHOLE, J5 8PIN2.54MM2X4TH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

Commit message: Revision A of the PCB is done
Parts:
- J8: value 10PIN2.54MM2X5TH -> 6PIN2.54MM2X3TH; device Headers:10PIN2.54MM2X5TH -> Headers:6PIN2.54MM2X3TH
Connections:
- net PA10: now also J8.3; no longer J8.7
- net PA12: now also J8.4; no longer J8.8
- net PA13: now also J8.5; no longer J8.9
- net PA14: now also J8.6; no longer J8.10
- net PA5: now also J8.2; no longer J8.6
- net PC7: no longer J9.13
- net PD16: no longer J8.2
- net PD18: no longer J8.3
- net PD19: no longer J8.4
- net PD22: no longer J8.5
Changed lines of the file:
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@@
 <part name="LED6" library="Semiconductors" deviceset="LED" device="1206"/>
 <part name="GND45" library="supply1" deviceset="GND" device=""/>
-<part name="J8" library="Headers" deviceset="10PIN" device="2.54MM2X5TH"/>
 <part name="LED7" library="Semiconductors" deviceset="LED" device="1206"/>
 <part name="R50" library="passives" deviceset="R" device="0603" value="330R"/>
@@
 <part name="J9" library="Headers" deviceset="16PIN" device="2.54MM2X8TH"/>
 <part name="GND47" library="supply1" deviceset="GND" device=""/>
+<part name="J8" library="Headers" deviceset="6PIN" device="2.54MM2X3TH"/>
 </parts>
 <sheets>
@@
 <instance part="LED6" gate="G$1" x="55.88" y="45.72"/>
 <instance part="GND45" gate="1" x="55.88" y="27.94" rot="MR0"/>
-<instance part="J8" gate="G$1" x="15.24" y="81.28" rot="R90"/>
 <instance part="J9" gate="G$1" x="33.02" y="81.28" rot="R90"/>
 <instance part="GND47" gate="1" x="78.74" y="33.02" rot="MR0"/>
+<instance part="J8" gate="G$1" x="12.7" y="81.28" rot="R90"/>
 </instances>
 <busses>
@@
 <net name="PA5" class="0">
 <segment>
-<pinref part="J8" gate="G$1" pin="6"/>
 <wire x1="20.32" y1="96.52" x2="20.32" y2="88.9" width="0.1524" layer="91"/>
 <label x="20.32" y="88.9" size="1.778" layer="95" rot="R90"/>
+<wire x1="20.32" y1="88.9" x2="20.32" y2="73.66" width="0.1524" layer="91"/>
+<wire x1="20.32" y1="73.66" x2="17.78" y2="71.12" width="0.1524" layer="91"/>
+<pinref part="J8" gate="G$1" pin="2"/>
+<wire x1="17.78" y1="71.12" x2="15.24" y2="71.12" width="0.1524" layer="91"/>
+<wire x1="15.24" y1="71.12" x2="12.7" y2="73.66" width="0.1524" layer="91"/>
 </segment>
 </net>
 <net name="PA10" class="0">
 <segment>
-<pinref part="J8" gate="G$1" pin="7"/>
 <wire x1="17.78" y1="88.9" x2="17.78" y2="96.52" width="0.1524" layer="91"/>
 <label x="17.78" y="88.9" size="1.778" layer="95" rot="R90"/>
+<wire x1="17.78" y1="88.9" x2="17.78" y2="88.138" width="0.1524" layer="91"/>
+<wire x1="17.78" y1="88.138" x2="19.304" y2="86.614" width="0.1524" layer="91"/>
+<wire x1="19.304" y1="86.614" x2="19.304" y2="75.184" width="0.1524" layer="91"/>
+<wire x1="19.304" y1="75.184" x2="18.034" y2="73.914" width="0.1524" layer="91"/>
+<wire x1="18.034" y1="73.914" x2="15.494" y2="73.914" width="0.1524" layer="91"/>
+<wire x1="15.494" y1="73.914" x2="15.24" y2="74.168" width="0.1524" layer="91"/>
+<pinref part="J8" gate="G$1" pin="3"/>
+<wire x1="15.24" y1="74.168" x2="15.24" y2="73.66" width="0.1524" layer="91"/>
 </segment>
 </net>
 <net name="PA12" class="0">
 <segment>
-<pinref part="J8" gate="G$1" pin="8"/>
 <wire x1="15.24" y1="88.9" x2="15.24" y2="96.52" width="0.1524" layer="91"/>
 <label x="15.24" y="88.9" size="1.778" layer="95" rot="R90"/>
+<pinref part="J8" gate="G$1" pin="4"/>
 </segment>
 </net>
 <net name="PA13" class="0">
 <segment>
-<pinref part="J8" gate="G$1" pin="9"/>
 <wire x1="12.7" y1="88.9" x2="12.7" y2="96.52" width="0.1524" layer="91"/>
 <label x="12.7" y="88.9" size="1.778" layer="95" rot="R90"/>
+<pinref part="J8" gate="G$1" pin="5"/>
 </segment>
 </net>
 <net name="PA14" class="0">
 <segment>
-<pinref part="J8" gate="G$1" pin="10"/>
 <wire x1="10.16" y1="88.9" x2="10.16" y2="96.52" width="0.1524" layer="91"/>
 <label x="10.16" y="88.9" size="1.778" layer="95" rot="R90"/>
+<pinref part="J8" gate="G$1" pin="6"/>
 </segment>
 </net>
@@
 </segment>
 </net>
-<net name="PC7" class="0">
-<segment>
-<pinref part="J9" gate="G$1" pin="13"/>
-<wire x1="33.02" y1="88.9" x2="33.02" y2="93.98" width="0.1524" layer="91"/>
-<label x="33.02" y="88.9" size="1.778" layer="95" rot="R90"/>
-</segment>
-</net>
 <net name="PC9" class="0">
 <segment>
@@
 <net name="PD4" class="0">
 <segment>
-<pinref part="J8" gate="G$1" pin="1"/>
 <wire x1="10.16" y1="73.66" x2="10.16" y2="68.58" width="0.1524" layer="91"/>
 <label x="10.16" y="68.58" size="1.778" layer="95" rot="R90"/>
-</segment>
-</net>
-<net name="PD16" class="0">
-<segment>
-<pinref part="J8" gate="G$1" pin="2"/>
-<wire x1="12.7" y1="73.66" x2="12.7" y2="68.58" width="0.1524" layer="91"/>
-<label x="12.7" y="68.58" size="1.778" layer="95" rot="R90"/>
-</segment>
-</net>
-<net name="PD18" class="0">
-<segment>
-<pinref part="J8" gate="G$1" pin="3"/>
-<wire x1="15.24" y1="73.66" x2="15.24" y2="68.58" width="0.1524" layer="91"/>
-<label x="15.24" y="68.58" size="1.778" layer="95" rot="R90"/>
-</segment>
-</net>
-<net name="PD19" class="0">
-<segment>
-<pinref part="J8" gate="G$1" pin="4"/>
-<wire x1="17.78" y1="73.66" x2="17.78" y2="68.58" width="0.1524" layer="91"/>
-<label x="17.78" y="68.58" size="1.778" layer="95" rot="R90"/>
-</segment>
-</net>
-<net name="PD22" class="0">
-<segment>
-<pinref part="J8" gate="G$1" pin="5"/>
-<wire x1="20.32" y1="73.66" x2="20.32" y2="68.58" width="0.1524" layer="91"/>
-<label x="20.32" y="68.58" size="1.778" layer="95" rot="R90"/>
+<pinref part="J8" gate="G$1" pin="1"/>
 </segment>
 </net>

Commit message: Final PCB Layout. Accurate costings
Parts:
- removed R42, R43: 39R, passives:R0603
- renumbered LED1 to MOTOR, LED7 to POWER
Connections:
- removed net DATA_N: IC1.DM, R42.2
- removed net DATA_P: IC1.DP, R43.2
- net USB_N: now also IC1.DM; no longer R42.1
- net USB_P: now also IC1.DP; no longer R43.1
Changed lines of the file:
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@@
 <part name="+3V37" library="supply1" deviceset="+3V3" device=""/>
 <part name="J4" library="Headers" deviceset="1BY2" device="THROUGHHOLE"/>
-<part name="R42" library="passives" deviceset="R" device="0603" value="39R"/>
-<part name="R43" library="passives" deviceset="R" device="0603" value="39R"/>
 <part name="C31" library="passives" deviceset="C-EU" device="C0603" value="100n"/>
 <part name="D1" library="Semiconductors" deviceset="DIODE" device="SMD"/>
@@
 <part name="GND39" library="supply1" deviceset="GND" device=""/>
 <part name="J7" library="Headers" deviceset="1BY2" device="THROUGHHOLE"/>
-<part name="LED1" library="Semiconductors" deviceset="LED" device="1206"/>
+<part name="MOTOR" library="Semiconductors" deviceset="LED" device="1206"/>
 <part name="R45" library="passives" deviceset="R" device="0603" value="330R"/>
 <part name="GND41" library="supply1" deviceset="GND" device=""/>
@@
 <part name="LED6" library="Semiconductors" deviceset="LED" device="1206"/>
 <part name="GND45" library="supply1" deviceset="GND" device=""/>
-<part name="LED7" library="Semiconductors" deviceset="LED" device="1206"/>
+<part name="POWER" library="Semiconductors" deviceset="LED" device="1206"/>
 <part name="R50" library="passives" deviceset="R" device="0603" value="330R"/>
 <part name="GND46" library="supply1" deviceset="GND" device=""/>
@@
 <instance part="+3V26" gate="G$1" x="231.14" y="35.56"/>
 <instance part="+3V27" gate="G$1" x="144.78" y="2.54"/>
-<instance part="R42" gate="G$1" x="96.52" y="-12.7" smashed="yes" rot="R90">
-<attribute name="NAME" x="95.0214" y="-14.986" size="1.778" layer="95" rot="R90"/>
-<attribute name="VALUE" x="96.266" y="-9.906" size="1.778" layer="96" rot="R90"/>
-</instance>
-<instance part="R43" gate="G$1" x="99.06" y="-12.7" smashed="yes" rot="R90">
-<attribute name="NAME" x="102.1334" y="-14.986" size="1.778" layer="95" rot="R90"/>
-<attribute name="VALUE" x="98.806" y="-9.906" size="1.778" layer="96" rot="R90"/>
-</instance>
 <instance part="C31" gate="G$1" x="238.76" y="88.9"/>
 <instance part="D1" gate="G$1" x="238.76" y="101.6"/>
 <instance part="+3V38" gate="G$1" x="238.76" y="110.49"/>
 <instance part="GND37" gate="1" x="238.76" y="81.28"/>
-<instance part="LED7" gate="G$1" x="236.22" y="139.7"/>
+<instance part="POWER" gate="G$1" x="236.22" y="139.7"/>
 <instance part="R50" gate="G$1" x="236.22" y="129.54" rot="R90"/>
 <instance part="GND46" gate="1" x="236.22" y="121.92"/>
@@
 </segment>
 <segment>
-<pinref part="LED7" gate="G$1" pin="A"/>
+<pinref part="POWER" gate="G$1" pin="A"/>
 <pinref part="+3V21" gate="G$1" pin="+3V3"/>
 </segment>
@@
 </segment>
 <segment>
-<pinref part="R43" gate="G$1" pin="1"/>
 <wire x1="99.06" y1="-17.78" x2="99.06" y2="-20.32" width="0.1524" layer="91"/>
 <label x="99.568" y="-19.812" size="1.778" layer="95"/>
+<pinref part="IC1" gate="G$1" pin="DP"/>
+<wire x1="99.06" y1="-5.08" x2="99.06" y2="-7.62" width="0.1524" layer="91"/>
+<wire x1="99.06" y1="-17.78" x2="99.06" y2="-7.62" width="0.1524" layer="91"/>
 </segment>
 </net>
@@
 </segment>
 <segment>
-<pinref part="R42" gate="G$1" pin="1"/>
 <wire x1="96.52" y1="-17.78" x2="96.52" y2="-20.32" width="0.1524" layer="91"/>
 <label x="96.52" y="-17.78" size="1.778" layer="95" rot="R180"/>
+<pinref part="IC1" gate="G$1" pin="DM"/>
+<wire x1="96.52" y1="-5.08" x2="96.52" y2="-7.62" width="0.1524" layer="91"/>
+<wire x1="96.52" y1="-17.78" x2="96.52" y2="-7.62" width="0.1524" layer="91"/>
 </segment>
 </net>
@@
 </segment>
 </net>
-<net name="DATA_N" class="0">
-<segment>
-<pinref part="IC1" gate="G$1" pin="DM"/>
-<pinref part="R42" gate="G$1" pin="2"/>
-<wire x1="96.52" y1="-5.08" x2="96.52" y2="-7.62" width="0.1524" layer="91"/>
-</segment>
-</net>
-<net name="DATA_P" class="0">
-<segment>
-<pinref part="IC1" gate="G$1" pin="DP"/>
-<pinref part="R43" gate="G$1" pin="2"/>
-<wire x1="99.06" y1="-5.08" x2="99.06" y2="-7.62" width="0.1524" layer="91"/>
-</segment>
-</net>
 <net name="N$36" class="0">
 <segment>
-<pinref part="LED7" gate="G$1" pin="C"/>
+<pinref part="POWER" gate="G$1" pin="C"/>
 <pinref part="R50" gate="G$1" pin="2"/>
 </segment>
@@
 <instance part="+3V34" gate="G$1" x="127" y="15.24" rot="MR0"/>
 <instance part="+3V35" gate="G$1" x="106.68" y="15.24" rot="MR0"/>
-<instance part="LED1" gate="G$1" x="71.12" y="55.88"/>
+<instance part="MOTOR" gate="G$1" x="71.12" y="55.88"/>
 <instance part="R45" gate="G$1" x="71.12" y="43.18" rot="R90"/>
 <instance part="GND41" gate="1" x="71.12" y="35.56"/>
@@
 <net name="N$31" class="0">
 <segment>
-<pinref part="LED1" gate="G$1" pin="C"/>
+<pinref part="MOTOR" gate="G$1" pin="C"/>
 <pinref part="R45" gate="G$1" pin="2"/>
 <wire x1="71.12" y1="50.8" x2="71.12" y2="48.26" width="0.1524" layer="91"/>
@@
 <net name="PB12" class="0">
 <segment>
-<pinref part="LED1" gate="G$1" pin="A"/>
+<pinref part="MOTOR" gate="G$1" pin="A"/>
 <wire x1="71.12" y1="63.5" x2="71.12" y2="58.42" width="0.1524" layer="91"/>
 <label x="71.12" y="60.96" size="1.778" layer="95"/>
